File: PHABB.kicad_pcb (KiCad board)
At the start: 2 copper layers, 102.5 x 77.5 mm, 88 parts, among them J1 RPi_GPIO, J2 SPI_SEL, J3 Inputs, J4 Vload, P25 GPIO2, U1 MCP3008, U2 LM2902, U3 LM2902

Commit message: add ID text for rev 1.0
Other:
- board text added: "Paul Hirst <contact@phirst.org> https://github.com/paulhirst/pi_filtered_adc_board R-Pi 8-channel Low-Pass Filtered ADC board Rev: 1.0"
Changed lines of the file:
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@@
+		)
+	)
+	(gr_text "Paul Hirst <contact@phirst.org>\nhttps://github.com/paulhirst/pi_filtered_adc_board\nR-Pi 8-channel Low-Pass Filtered ADC board\nRev: 1.0"
+		(at 72.67 89 90)
+		(layer "F.SilkS")
+		(effects
+			(font
+				(size 1 1)
+				(thickness 0.1)
+			)
+			(justify left bottom)
 		)
 	)
